Commit message: Update rail and positioner launch files and urdf macros

File: twc_support/CAD/rail/gudel_tmf2/urdf/gudel_tmf2_dual_macro.xacro (robot description, xacro)
@@ -1,5 +1,5 @@
 <?xml version="1.0"?>
 <robot xmlns:xacro="http://wiki.ros.org/xacro">
-  <xacro:macro name="gudel_tmf2_dual" params="prefix">
+  <xacro:macro name="gudel_tmf2_dual" params="prefix length">
     <!-- link list -->
     <link name="${prefix}base_link">
@@ -7,5 +7,13 @@
         <origin xyz="0 0 0" rpy="0 0 0" />
         <geometry>
-          <mesh filename="package://twc_support/CAD/rail/gudel_tmf2/urdf/visual/base_link.dae" />
+          <xacro:if value="${length == 5}">
+            <mesh filename="package://twc_support/CAD/rail/gudel_tmf2/urdf/visual/base_link_05m.dae" />
+          </xacro:if>
+          <xacro:if value="${length == 10}">
+            <mesh filename="package://twc_support/CAD/rail/gudel_tmf2/urdf/visual/base_link_10m.dae" />
+          </xacro:if>
+          <xacro:if value="${length == 12}">
+            <mesh filename="package://twc_support/CAD/rail/gudel_tmf2/urdf/visual/base_link_12m.dae" />
+          </xacro:if>
         </geometry>
       </visual>
@@ -13,5 +21,13 @@
         <origin xyz="0 0 0" rpy="0 0 0" />
         <geometry>
-          <mesh filename="package://twc_support/CAD/rail/gudel_tmf2/urdf/visual/base_link.dae" />
+          <xacro:if value="${length == 5}">
+            <mesh filename="package://twc_support/CAD/rail/gudel_tmf2/urdf/visual/base_link_05m.dae" />
+          </xacro:if>
+          <xacro:if value="${length == 10}">
+            <mesh filename="package://twc_support/CAD/rail/gudel_tmf2/urdf/visual/base_link_10m.dae" />
+          </xacro:if>
+          <xacro:if value="${length == 12}">
+            <mesh filename="package://twc_support/CAD/rail/gudel_tmf2/urdf/visual/base_link_12m.dae" />
+          </xacro:if>
         </geometry>
       </collision>

File: twc_support/CAD/rail/gudel_tmf2/urdf/gudel_tmf2_single_macro.xacro (robot description, xacro)
@@ -1,5 +1,5 @@
 <?xml version="1.0"?>
 <robot xmlns:xacro="http://wiki.ros.org/xacro">
-  <xacro:macro name="gudel_tmf2_single" params="prefix">
+  <xacro:macro name="gudel_tmf2_single" params="prefix length">
     <!-- link list -->
     <link name="${prefix}base_link">
@@ -7,5 +7,13 @@
         <origin xyz="0 0 0" rpy="0 0 0" />
         <geometry>
-          <mesh filename="package://twc_support/CAD/rail/gudel_tmf2/urdf/visual/base_link.dae" />
+          <xacro:if value="${length == 5}">
+            <mesh filename="package://twc_support/CAD/rail/gudel_tmf2/urdf/visual/base_link_05m.dae" />
+          </xacro:if>
+          <xacro:if value="${length == 10}">
+            <mesh filename="package://twc_support/CAD/rail/gudel_tmf2/urdf/visual/base_link_10m.dae" />
+          </xacro:if>
+          <xacro:if value="${length == 12}">
+            <mesh filename="package://twc_support/CAD/rail/gudel_tmf2/urdf/visual/base_link_12m.dae" />
+          </xacro:if>
         </geometry>
       </visual>
@@ -13,5 +21,13 @@
         <origin xyz="0 0 0" rpy="0 0 0" />
         <geometry>
-          <mesh filename="package://twc_support/CAD/rail/gudel_tmf2/urdf/visual/base_link.dae" />
+          <xacro:if value="${length == 5}">
+            <mesh filename="package://twc_support/CAD/rail/gudel_tmf2/urdf/visual/base_link_05m.dae" />
+          </xacro:if>
+          <xacro:if value="${length == 10}">
+            <mesh filename="package://twc_support/CAD/rail/gudel_tmf2/urdf/visual/base_link_10m.dae" />
+          </xacro:if>
+          <xacro:if value="${length == 12}">
+            <mesh filename="package://twc_support/CAD/rail/gudel_tmf2/urdf/visual/base_link_12m.dae" />
+          </xacro:if>
         </geometry>
       </collision>
@@ -35,9 +51,9 @@
     <!-- joint list -->
     <joint name="${prefix}joint_1" type="prismatic">
-      <origin xyz="0 0 0" rpy="0 0 0" />
+      <origin xyz="0 0.2 0" rpy="0 0 0" />
       <parent link="${prefix}base_link" />
       <child link="${prefix}link_1" />
       <axis xyz="0 1 0" />
-      <limit lower="0" upper="10" effort="0" velocity="2.5" />
+      <limit lower="0" upper="${length - 1}" effort="0" velocity="2.5" />
     </joint>
     <joint name="${prefix}joint_1_tool0" type="fixed">

File: twc_support/urdf/workcell_rail.urdf (robot description, URDF)
Before this commit: robot tesseract_workcell_rail, 45 links, 44 joints
Links:
- removed link fence_panel4_base_link
- removed link fence_panel4_tool0
- removed link fence_panel5_base_link
- removed link fence_panel5_tool0
- removed link fence_panel6_base_link
- removed link fence_panel6_tool0
- removed link fence_panel7_base_link
- removed link fence_panel7_tool0
- link rail_base_link: geometry 
Joints:
- removed joint fence_panel4_joint
- removed joint fence_panel4_joint_1
- removed joint fence_panel5_joint
- removed joint fence_panel5_joint_1
- removed joint fence_panel6_joint
- removed joint fence_panel6_joint_1
- removed joint fence_panel7_joint
- removed joint fence_panel7_joint_1

File: twc_support/urdf/workcell_rail_macro.xacro (robot description, xacro)
@@ -17,13 +17,9 @@
     <xacro:abb_irb4600_60_205 prefix="robot_"/>
     <xacro:include filename="$(find twc_support)/CAD/rail/gudel_tmf2/urdf/gudel_tmf2_single_macro.xacro"/>
-    <xacro:gudel_tmf2_single prefix="rail_"/>
+    <xacro:gudel_tmf2_single prefix="rail_" length="5"/>
     <xacro:include filename="$(find twc_support)/CAD/fence/panel_3m_2m_solid/urdf/panel_3m_2m_solid_macro.xacro"/>
     <xacro:panel_3m_2m_solid prefix="fence_panel1_"/>
     <xacro:panel_3m_2m_solid prefix="fence_panel2_"/>
     <xacro:panel_3m_2m_solid prefix="fence_panel3_"/>
-    <xacro:panel_3m_2m_solid prefix="fence_panel4_"/>
-    <xacro:panel_3m_2m_solid prefix="fence_panel5_"/>
-    <xacro:panel_3m_2m_solid prefix="fence_panel6_"/>
-    <xacro:panel_3m_2m_solid prefix="fence_panel7_"/>
     <xacro:include filename="$(find twc_support)/CAD/logo/ros_industrial/urdf/ros_industrial_logo_macro.xacro"/>
     <xacro:ros_industrial_logo prefix="logo_"/>
@@ -51,9 +47,9 @@
       <child link="${prefix}positioner_base_link" />
     </joint>
-  <joint name="${prefix}world_rail_joint" type="fixed">
-    <origin xyz="6 -1 0" rpy="0 0 1.5708" />
-    <parent link="${prefix}world" />
-    <child link="${prefix}rail_base_link" />
-  </joint>
+    <joint name="${prefix}world_rail_joint" type="fixed">
+      <origin xyz="2.5 -1 0" rpy="0 0 1.5708" />
+      <parent link="${prefix}world" />
+      <child link="${prefix}rail_base_link" />
+    </joint>
     <joint name="${prefix}rail_robot_joint" type="fixed">
       <origin xyz="0 0 0" rpy="0 0 0" />
@@ -104,5 +100,5 @@
     </joint>
     <joint name="${prefix}fence_panel1_joint" type="fixed">
-      <origin xyz="-7 -2 0" rpy="0 0 0" />
+      <origin xyz="-3 -2 0" rpy="0 0 0" />
       <parent link="${prefix}world" />
       <child link="${prefix}fence_panel1_base_link" />
@@ -118,24 +114,4 @@
       <child link="${prefix}fence_panel3_base_link" />
     </joint>
-    <joint name="${prefix}fence_panel4_joint" type="fixed">
-      <origin xyz="0 0 0" rpy="0 0 0" />
-      <parent link="${prefix}fence_panel3_tool0" />
-      <child link="${prefix}fence_panel4_base_link" />
-    </joint>
-    <joint name="${prefix}fence_panel5_joint" type="fixed">
-      <origin xyz="0 0 0" rpy="0 0 0" />
-      <parent link="${prefix}fence_panel4_tool0" />
-      <child link="${prefix}fence_panel5_base_link" />
-    </joint>
-    <joint name="${prefix}fence_panel6_joint" type="fixed">
-      <origin xyz="0 0 0" rpy="0 0 0" />
-      <parent link="${prefix}fence_panel5_tool0" />
-      <child link="${prefix}fence_panel6_base_link" />
-    </joint>
-    <joint name="${prefix}fence_panel7_joint" type="fixed">
-      <origin xyz="0 0 0" rpy="0 0 0" />
-      <parent link="${prefix}fence_panel6_tool0" />
-      <child link="${prefix}fence_panel7_base_link" />
-    </joint>
     <joint name="${prefix}logo_joint" type="fixed">
       <origin xyz="0.9 0 2.3" rpy="1.5708 0 3.14159" />
