Commit message: Add offset tool0 link to bt30 sander urdf

File: twc_support/CAD/eoat/bt30_sander/urdf/bt30_sander_macro.xacro (robot description, xacro)
@@ -18,4 +18,5 @@
     </link>
     <link name="${prefix}tool0"/>
+    <link name="${prefix}tool0_offset"/>
     <!-- end of link list -->
     <!-- joint list -->
@@ -25,4 +26,9 @@
       <child link="${prefix}tool0" />
     </joint>
+    <joint name="${prefix}joint_tool0_offset" type="fixed">
+      <origin xyz="0 0 0.05" rpy="0 0 0" />
+      <parent link="${prefix}tool0" />
+      <child link="${prefix}tool0_offset" />
+    </joint>
     <!-- end of joint list -->
   </xacro:macro>

Commit message: fixup

File: twc_support/CAD/eoat/bt30_sander/urdf/bt30_sander_macro.xacro (robot description, xacro)
@@ -3,5 +3,6 @@
   <xacro:macro name="bt30_sander" params="prefix">
     <!-- link list -->
-    <link name="${prefix}base_link">
+    <link name="${prefix}base_link"/>
+    <link name="${prefix}sander_link">
       <visual>
         <origin xyz="0 0 0" rpy="0 0 0" />
@@ -20,8 +21,20 @@
     <link name="${prefix}tool0_offset"/>
     <!-- end of link list -->
+    <xacro:include filename="$(find twc_support)/CAD/eoat/bt30/urdf/bt30_macro.xacro"/>
+    <xacro:bt30 prefix="${prefix}bt_"/>
     <!-- joint list -->
+    <joint name="${prefix}joint_bt30" type="fixed">
+      <origin xyz="0 0 0" rpy="0 0 0" />
+      <parent link="${prefix}base_link" />
+      <child link="${prefix}bt_base_link" />
+    </joint>
+    <joint name="${prefix}joint_sander" type="fixed">
+      <origin xyz="0 0 0" rpy="0 0 0" />
+      <parent link="${prefix}bt_tool0" />
+      <child link="${prefix}sander_link" />
+    </joint>
     <joint name="${prefix}joint_tool0" type="fixed">
-      <origin xyz="0 0 0.07328" rpy="0 0 0" />
-      <parent link="${prefix}base_link" />
+      <origin xyz="0 0 0.0253" rpy="0 0 0" />
+      <parent link="${prefix}sander_link" />
       <child link="${prefix}tool0" />
     </joint>
